File: tp60.sch (KiCad schematic (older format))
At the start: 126 parts, among them J1 Conn_01x10_MountingPin, K1 KEYSW, K10 KEYSW, K11 KEYSW, K12 KEYSW, K13 KEYSW, K14 KEYSW, K15 KEYSW, K16 KEYSW, K17 KEYSW, K18 KEYSW, K19 KEYSW, K2 KEYSW, K20 KEYSW, K21 KEYSW, K22 KEYSW, K23 KEYSW, K24 KEYSW, K25 KEYSW, K26 KEYSW, K27 KEYSW, K28 KEYSW, K29 KEYSW, K3 KEYSW, K30 KEYSW, K31 KEYSW, K32 KEYSW, K33 KEYSW, K34 KEYSW, K35 KEYSW, K36 KEYSW, K37 KEYSW, K38 KEYSW, K39 KEYSW, K4 KEYSW, K40 KEYSW, K41 KEYSW, K42 KEYSW, K43 KEYSW, K44 KEYSW, K45 KEYSW, K46 KEYSW, K47 KEYSW, K48 KEYSW, K49 KEYSW, K5 KEYSW, K50 KEYSW, K51 KEYSW, K52 KEYSW, K53 KEYSW, K54 KEYSW, K55 KEYSW, K56 KEYSW, K57 KEYSW, K58 KEYSW, K59 KEYSW, K6 KEYSW, K7 KEYSW, K8 KEYSW, K9 KEYSW, P1 CONN_5, P2 CONN_4, P3 CONN_5, P4 CONN_4, P5 CONN_4, P6 CONN_10, P7 CONN_8

Commit message: refilled zone
Changed lines of the file:
@@
 L power:PWR_FLAG #FLG0101
 U 1 1 5EB2B625
-P 2950 8900
-F 0 "#FLG0101" H 2950 8975 50  0001 C CNN
-F 1 "PWR_FLAG" V 2950 9027 50  0000 L CNN
-F 2 "" H 2950 8900 50  0001 C CNN
-F 3 "~" H 2950 8900 50  0001 C CNN
-	1    2950 8900
-	0    -1   -1   0
+P 2650 8900
+F 0 "#FLG0101" H 2650 8975 50  0001 C CNN
+F 1 "PWR_FLAG" V 2650 9027 50  0000 L CNN
+F 2 "" H 2650 8900 50  0001 C CNN
+F 3 "~" H 2650 8900 50  0001 C CNN
+	1    2650 8900
+	-1   0    0    1
 $EndComp
 Wire Wire Line
 	2950 8900 2650 8900
+Connection ~ 2650 8900
 $EndSCHEMATC

Commit message: rewrite pcb
Parts:
- K1, K10, K11, K12, K13, K14, K15, K16, K17, K18, K19, K2, K20, K21, K22, K23, K24, K25, K26, K27, K28, K29, K3, K30, K31, K32, K33, K34, K35, K36, K37, K38, K39, K4, K40, K41, K42, K43, K44, K45, K46, K47, K48, K49, K5, K50, K51, K52, K53, K54, K55, K56, K57, K58, K59, K6, K7, K8, K9: footprint keyswitches:Kailh_socket_MX_optional_r -> keyswitches:SW_MX_1280
Other:
- moved on the sheet: K1, K10, K11, K12, K13, K14, K15, K16, K17, K18, K19, K2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

Commit message: improved pcb lines
Parts:
- added SW1: SW_PUSH, Button_Switch_SMD:SW_Push_1P1T_NO_6x6mm_H9.5mm, symbol keyboard_parts:SW_PUSH
- P1: value CONN_5 -> CONN_6; footprint Connector_PinHeader_2.54mm:PinHeader_1x05_P2.54mm_Vertical -> Connector_PinHeader_2.54mm:PinHeader_1x06_P2.54mm_Vertical; symbol conn:CONN_5 -> conn:CONN_6
- P5: footprint Connector_PinHeader_2.54mm:PinHeader_1x04_P2.54mm_Vertical -> Connector_PinHeader_2.54mm:PinHeader_2x05_P2.54mm_Vertical; symbol conn:CONN_4 -> conn:CONN_5X2
- P6: footprint Connector_PinSocket_2.54mm:PinSocket_1x10_P2.54mm_Vertical -> Connector_PinHeader_2.54mm:PinHeader_2x05_P2.54mm_Vertical
- P7: footprint Connector_USB:USB_C_Receptacle_Palconn_UTC16-G -> Type-C:HRO-TYPE-C-31-M-12-PIN; symbol Connector:USB_C_Plug_USB2.0 -> Connector:USB_C_Receptacle_USB2.0
Connections:
- wire segments 154 -> 188
- no-connect marks 4 -> 1
Other:
- note added: "TP60"
- moved on the sheet: K10, K11, K2, K26, K3, K37, K4, K5, K52, K53, K54, K55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
