File: tp60.kicad_pcb (KiCad board)
At the start: 2 copper layers, 285.3 x 94.9 mm, 127 parts, among them J1 Conn_01x10_MountingPin, K1 KEYSW, K10 KEYSW, K11 KEYSW, K12 KEYSW, K13 KEYSW, K14 KEYSW, K15 KEYSW, K16 KEYSW, K17 KEYSW, K18 KEYSW, K19 KEYSW, K2 KEYSW, K20 KEYSW, K21 KEYSW, K22 KEYSW, K23 KEYSW, K24 KEYSW, K25 KEYSW, K26 KEYSW, K27 KEYSW, K28 KEYSW, K29 KEYSW, K3 KEYSW, K30 KEYSW, K31 KEYSW, K32 KEYSW, K33 KEYSW, K34 KEYSW, K35 KEYSW, K36 KEYSW, K37 KEYSW, K38 KEYSW, K39 KEYSW, K4 KEYSW, K40 KEYSW, K41 KEYSW, K42 KEYSW, K43 KEYSW, K44 KEYSW, K45 KEYSW, K46 KEYSW, K47 KEYSW, K48 KEYSW, K49 KEYSW, K5 KEYSW, K50 KEYSW, K51 KEYSW, K52 KEYSW, K53 KEYSW, K54 KEYSW, K55 KEYSW, K56 KEYSW, K57 KEYSW, K58 KEYSW, K59 KEYSW, K6 KEYSW, K7 KEYSW, K8 KEYSW, K9 KEYSW, P1 CONN_5, P2 CONN_4, P3 CONN_5, P4 CONN_4, P5 CONN_4, P6 CONN_10, P7 CONN_8

Commit message: refilled zone
Parts:
- removed G***: oshw_logo, logos:oshw
- added REF**: OSHW-Logo2_14.6x12mm_SilkScreen, Symbol:OSHW-Logo2_14.6x12mm_SilkScreen, F.Cu at (343.0, 176.0)
- moved D44 5.06 mm to (201.3, 157.5)
- moved D1 0.30 mm to (91.0, 110.5)
Routing:
- net /row1: track 273.1 -> 296.8 mm
- net +5V: track 20.1 -> 13.6 mm
- net /col06: track 137.8 -> 142.5 mm
- net Net-(D1-Pad2): track 16.2 -> 12.3 mm
- net Net-(D44-Pad2): track 13.1 -> 11.3 mm
- net /row4: track 359.0 -> 360.7 mm
- net /col01: track 163.3 -> 164.8 mm
- net /row3: track 358.1 -> 359.0 mm
- added copper zone on B.Cu, net GND
- removed copper zone on B.Cu, net Net-(J1-Pad7)
Other:
- outline, holes or cut-outs redrawn

Commit message: rewrite pcb
Parts:
- removed the REF** at (343.0, 176.0)
- added REF**: OSHW-Symbol_8.9x8mm_SilkScreen, Symbol:OSHW-Symbol_8.9x8mm_SilkScreen, F.Cu at (342.0, 175.3)
- K1, K10, K11, K12, K13, K14, K15, K16, K17, K18, K19, K2, K20, K21, K22, K23, K24, K25, K26, K27, K28, K29, K3, K30, K31, K32, K33, K34, K35, K36, K37, K38, K39, K4, K40, K41, K42, K43, K44, K45, K46, K47, K48, K49, K5, K50, K51, K52, K53, K54, K55, K56, K57, K58, K59, K6, K7, K8, K9: footprint keyswitches:Kailh_socket_MX_optional_r -> keyswitches:SW_MX_1280
- moved P3 7.60 mm to (204.9, 169.6)
- moved D51 4.70 mm to (90.8, 169.0)
- moved D59 4.40 mm to (329.4, 169.0)
- moved P5 1.95 mm to (78.0, 108.7)
- moved D44 1.13 mm to (200.5, 156.7)
- moved P6 0.68 mm to (342.2, 130.2)
- moved J1 0.68 mm to (343.3, 105.4)
- turned K26 to 0 degrees
- turned K27 to 0 degrees
- turned K28 to 0 degrees
- turned K29 to 0 degrees
- turned K30 to 0 degrees
- turned K31 to 0 degrees
- turned K32 to 0 degrees
- turned K33 to 0 degrees
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Connections:
- K1 pad 1: /col01 -> Net-(D1-Pad2)
- K1 pad 2: Net-(D1-Pad2) -> /col01
- K10 pad 1: Net-(D10-Pad2) -> /col11
- K10 pad 2: /col11 -> Net-(D10-Pad2)
- K11 pad 1: Net-(D11-Pad2) -> /col12
- K11 pad 2: /col12 -> Net-(D11-Pad2)
- K12 pad 1: Net-(D12-Pad2) -> /col13
- K12 pad 2: /col13 -> Net-(D12-Pad2)
- K13 pad 1: Net-(D13-Pad2) -> /col01
- K13 pad 2: /col01 -> Net-(D13-Pad2)
- K14 pad 1: Net-(D14-Pad2) -> /col02
- K14 pad 2: /col02 -> Net-(D14-Pad2)
- K15 pad 1: Net-(D15-Pad2) -> /col03
- K15 pad 2: /col03 -> Net-(D15-Pad2)
- K16 pad 1: Net-(D16-Pad2) -> /col04
- K16 pad 2: /col04 -> Net-(D16-Pad2)
- K17 pad 1: Net-(D17-Pad2) -> /col05
- K17 pad 2: /col05 -> Net-(D17-Pad2)
- K18 pad 1: Net-(D18-Pad2) -> /col06
- K18 pad 2: /col06 -> Net-(D18-Pad2)
- K19 pad 1: Net-(D19-Pad2) -> /col07
- K19 pad 2: /col07 -> Net-(D19-Pad2)
- K2 pad 1: /col02 -> Net-(D2-Pad2)
- K2 pad 2: Net-(D2-Pad2) -> /col02
- K20 pad 1: /col08 -> Net-(D20-Pad2)
- K20 pad 2: Net-(D20-Pad2) -> /col08
- K21 pad 1: /col09 -> Net-(D21-Pad2)
- K21 pad 2: Net-(D21-Pad2) -> /col09
- K22 pad 1: /col10 -> Net-(D22-Pad2)
- K22 pad 2: Net-(D22-Pad2) -> /col10
- K23 pad 1: /col11 -> Net-(D23-Pad2)
- K23 pad 2: Net-(D23-Pad2) -> /col11
- K24 pad 1: /col12 -> Net-(D24-Pad2)
- K24 pad 2: Net-(D24-Pad2) -> /col12
- K25 pad 1: /col13 -> Net-(D25-Pad2)
- K25 pad 2: Net-(D25-Pad2) -> /col13
- K3 pad 1: /col03 -> Net-(D3-Pad2)
- K3 pad 2: Net-(D3-Pad2) -> /col03
- K4 pad 1: /col04 -> Net-(D4-Pad2)
- K4 pad 2: Net-(D4-Pad2) -> /col04
- K5 pad 1: /col05 -> Net-(D5-Pad2)
- K5 pad 2: Net-(D5-Pad2) -> /col05
- K6 pad 1: /col06 -> Net-(D6-Pad2)
- K6 pad 2: Net-(D6-Pad2) -> /col06
- K7 pad 1: Net-(D7-Pad2) -> /col08
- K7 pad 2: /col08 -> Net-(D7-Pad2)
- K8 pad 1: Net-(D8-Pad2) -> /col09
- K8 pad 2: /col09 -> Net-(D8-Pad2)
- K9 pad 1: Net-(D9-Pad2) -> /col10
- K9 pad 2: /col10 -> Net-(D9-Pad2)
Routing:
- net /col01: track 164.8 -> 117.7 mm
- net /col06: track 142.5 -> 106.1 mm
- net /col04: track 129.6 -> 96.6 mm
- net /col10: track 131.1 -> 99.6 mm
- net /row1: track 296.8 -> 272.8 mm
- net /col03: track 106.8 -> 83.7 mm
- net /col11: track 105.1 -> 83.5 mm
- net /col05: track 121.3 -> 102.1 mm
- net /col13: track 158.8 -> 144.0 mm
- net Net-(D59-Pad2): track 21.6 -> 8.40 mm
- net /col12: track 102.4 -> 90.1 mm
- net /col07: track 78.0 -> 66.3 mm
- net Net-(D51-Pad2): track 16.5 -> 5.98 mm
- net /col02: track 106.9 -> 96.7 mm
- net Net-(D57-Pad2): track 21.9 -> 13.0 mm
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Other:
- outline, holes or cut-outs redrawn
- net class PG: trace_width 0.5 -> 0.3
- rule via_min_size: 0.4 -> 0.3

Commit message: improved pcb lines
Parts:
- added SW1: SW_PUSH, Button_Switch_SMD:SW_Push_1P1T_NO_6x6mm_H9.5mm, B.Cu at (90.4, 138.4)
- P1: value CONN_5 -> CONN_6; footprint Connector_PinHeader_2.54mm:PinHeader_1x05_P2.54mm_Vertical -> Connector_PinHeader_2.54mm:PinHeader_1x06_P2.54mm_Vertical; moved to B.Cu
- P2, P4: moved to B.Cu
- P5: footprint Connector_PinHeader_2.54mm:PinHeader_1x04_P2.54mm_Vertical -> Connector_PinHeader_2.54mm:PinHeader_2x05_P2.54mm_Vertical; moved to B.Cu
- P6: footprint Connector_PinSocket_2.54mm:PinSocket_1x10_P2.54mm_Vertical -> Connector_PinHeader_2.54mm:PinHeader_2x05_P2.54mm_Vertical; moved to B.Cu
- P7: footprint Connector_USB:USB_C_Receptacle_Palconn_UTC16-G -> Type-C:HRO-TYPE-C-31-M-12-PIN
- moved D59 20.7 mm to (309.3, 174.0)
- moved D51 20.6 mm to (110.8, 174.0)
- moved D37 20.2 mm to (309.9, 143.5)
- moved D26 19.9 mm to (110.1, 143.5)
- moved D12 19.5 mm to (310.0, 108.0)
- moved D1 19.2 mm to (110.1, 108.0)
- moved D19 12.6 mm to (200.5, 127.0), turned to 90 degrees
- moved D16 12.6 mm to (143.3, 127.0), turned to 90 degrees
- moved D17 12.6 mm to (162.4, 127.0), turned to 90 degrees
- moved D18 12.6 mm to (181.5, 127.0), turned to 90 degrees
- moved D20 12.6 mm to (238.6, 127.0), turned to 90 degrees
- moved D21 12.6 mm to (257.7, 127.0), turned to 90 degrees
- moved D22 12.6 mm to (276.7, 127.0), turned to 90 degrees
- moved D23 12.6 mm to (295.7, 127.0), turned to 90 degrees
- moved D24 12.6 mm to (314.7, 127.0), turned to 90 degrees
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Connections:
- J1 pad MP: Net-(J1-PadMP) -> GND
- K10 pad 1: /col11 -> Net-(D10-Pad2)
- K10 pad 2: Net-(D10-Pad2) -> /col11
- K11 pad 1: /col12 -> Net-(D11-Pad2)
- K11 pad 2: Net-(D11-Pad2) -> /col12
- K2 pad 1: Net-(D2-Pad2) -> /col02
- K2 pad 2: /col02 -> Net-(D2-Pad2)
- K26 pad 1: /col01 -> Net-(D26-Pad2)
- K26 pad 2: Net-(D26-Pad2) -> /col01
- K3 pad 1: Net-(D3-Pad2) -> /col03
- K3 pad 2: /col03 -> Net-(D3-Pad2)
- K37 pad 1: Net-(D37-Pad2) -> /col13
- K37 pad 2: /col13 -> Net-(D37-Pad2)
- K4 pad 1: Net-(D4-Pad2) -> /col04
- K4 pad 2: /col04 -> Net-(D4-Pad2)
- K5 pad 1: Net-(D5-Pad2) -> /col05
- K5 pad 2: /col05 -> Net-(D5-Pad2)
- K52 pad 1: /col03 -> Net-(D52-Pad2)
- K52 pad 2: Net-(D52-Pad2) -> /col03
- K53 pad 1: /col04 -> Net-(D53-Pad2)
- K53 pad 2: Net-(D53-Pad2) -> /col04
- K54 pad 1: /col06 -> Net-(D54-Pad2)
- K54 pad 2: Net-(D54-Pad2) -> /col06
- K55 pad 1: /col07 -> Net-(D55-Pad2)
- K55 pad 2: Net-(D55-Pad2) -> /col07
- K56 pad 1: Net-(D56-Pad2) -> /col08
- K56 pad 2: /col08 -> Net-(D56-Pad2)
- K57 pad 1: Net-(D57-Pad2) -> /col10
- K57 pad 2: /col10 -> Net-(D57-Pad2)
- K58 pad 1: Net-(D58-Pad2) -> /col11
- K58 pad 2: /col11 -> Net-(D58-Pad2)
- K6 pad 1: Net-(D6-Pad2) -> /col06
- K6 pad 2: /col06 -> Net-(D6-Pad2)
- K7 pad 1: /col08 -> Net-(D7-Pad2)
- K7 pad 2: Net-(D7-Pad2) -> /col08
- K8 pad 1: /col09 -> Net-(D8-Pad2)
- K8 pad 2: Net-(D8-Pad2) -> /col09
- K9 pad 1: /col10 -> Net-(D9-Pad2)
- K9 pad 2: Net-(D9-Pad2) -> /col10
- P5 pad 1: +5V -> Net-(P5-Pad1)
- P5 pad 4: GND -> Net-(P5-Pad4)
- P7 pad A5: Net-(P7-PadA5) -> Net-(P5-Pad6)
- P7 pad A6: Net-(P5-Pad3) -> Net-(P5-Pad2)
- P7 pad A7: Net-(P5-Pad2) -> Net-(P5-Pad1)
- P7 pad A8: (no net) -> Net-(P5-Pad5)
- P7 pad B5: Net-(P7-PadB5) -> Net-(P5-Pad7)
- P7 pad B6: (no net) -> Net-(P5-Pad3)
- P7 pad B7: (no net) -> Net-(P5-Pad4)
- P7 pad B8: (no net) -> Net-(P5-Pad8)
Routing:
- net /row3: track 359.7 -> 233.4 mm
- net /row4: track 358.7 -> 266.3 mm
- net /col04: track 96.6 -> 131.7 mm
- net /col10: track 99.6 -> 132.2 mm
- net /col13: track 144.0 -> 116.6 mm
- net /row1: track 272.8 -> 245.8 mm
- net /row5: track 273.5 -> 249.5 mm
- net /col03: track 83.7 -> 104.7 mm
- net Net-(P1-Pad6): track 0.00 -> 20.2 mm
- net /col11: track 83.5 -> 103.3 mm
- net /col08: track 106.2 -> 124.8 mm
- net /row2: track 275.2 -> 261.2 mm
- net Net-(P5-Pad7): track 0.00 -> 13.7 mm
- net Net-(P5-Pad8): track 0.00 -> 13.7 mm
- net /col02: track 96.7 -> 84.1 mm
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Other:
- net class PG: trace_width 0.3 -> 0.4

Commit message: made up pcb img and README
Parts:
- removed the REF** at (342.0, 175.3)
- added REF**: OSHW-Logo2_9.8x8mm_SilkScreen, Symbol:OSHW-Logo2_9.8x8mm_SilkScreen, F.Cu at (341.9, 176.0)

Commit message: adjusted socket pos
Parts:
- moved SW1 10.2 mm to (96.0, 146.9), turned to 180 degrees
- moved P6 2.17 mm to (344.5, 134.7)
- moved J1 1.57 mm to (344.3, 104.1)
- moved P7 1.10 mm to (85.8, 92.0)
- moved P5 0.45 mm to (87.1, 105.1)
Routing:
- net Net-(P1-Pad6): track 20.2 -> 14.8 mm
- net Net-(P5-Pad8): track 13.7 -> 14.9 mm
- net /col02: track 84.1 -> 82.9 mm
- net Net-(P5-Pad6): track 10.9 -> 12.1 mm
- net Net-(P5-Pad5): track 10.9 -> 12.1 mm
- net Net-(P5-Pad7): track 13.7 -> 14.8 mm
- net Net-(J1-Pad2): track 32.5 -> 31.4 mm
- net Net-(P5-Pad3): track 8.17 -> 9.29 mm
- net Net-(P5-Pad4): track 8.16 -> 9.27 mm
- net Net-(P5-Pad2): track 4.84 -> 5.84 mm
- net Net-(P5-Pad1): track 4.84 -> 5.84 mm
- net +5V: track 24.2 -> 25.1 mm
Other:
- outline, holes or cut-outs redrawn
